Commit message: Kinda working

File: dragon_long.urdf (robot description, URDF)
Before this commit: robot L1, 54 links, 53 joints
Joints:
- joint L1_vec_theta: limit lower=-1.57 upper=1.57 effort=5 velocity=2 -> lower=-3.14 upper=3.14 effort=5 velocity=2
- joint L2_vec_theta: limit lower=-1.57 upper=1.57 effort=5 velocity=2 -> lower=-3.14 upper=3.14 effort=5 velocity=2
- joint L3_vec_theta: limit lower=-1.57 upper=1.57 effort=5 velocity=2 -> lower=-3.14 upper=3.14 effort=5 velocity=2
- joint L4_vec_theta: limit lower=-1.57 upper=1.57 effort=5 velocity=2 -> lower=-3.14 upper=3.14 effort=5 velocity=2
- joint L5_vec_theta: limit lower=-1.57 upper=1.57 effort=5 velocity=2 -> lower=-3.14 upper=3.14 effort=5 velocity=2
- joint L6_vec_theta: limit lower=-1.57 upper=1.57 effort=5 velocity=2 -> lower=-3.14 upper=3.14 effort=5 velocity=2
- joint L7_vec_theta: limit lower=-1.57 upper=1.57 effort=5 velocity=2 -> lower=-3.14 upper=3.14 effort=5 velocity=2
- joint L8_vec_theta: limit lower=-1.57 upper=1.57 effort=5 velocity=2 -> lower=-3.14 upper=3.14 effort=5 velocity=2
- joint joint1_pitch: limit lower=-1.57 upper=1.57 effort=10 velocity=2 -> lower=-3.14 upper=3.14 effort=10 velocity=2
- joint joint1_yaw: limit lower=-1.57 upper=1.57 effort=10 velocity=2 -> lower=-3.14 upper=3.14 effort=10 velocity=2
- joint joint2_pitch: limit lower=-1.57 upper=1.57 effort=10 velocity=2 -> lower=-3.14 upper=3.14 effort=10 velocity=2
- joint joint2_yaw: limit lower=-1.57 upper=1.57 effort=10 velocity=2 -> lower=-3.14 upper=3.14 effort=10 velocity=2
- joint joint3_pitch: limit lower=-1.57 upper=1.57 effort=10 velocity=2 -> lower=-3.14 upper=3.14 effort=10 velocity=2
- joint joint3_yaw: limit lower=-1.57 upper=1.57 effort=10 velocity=2 -> lower=-3.14 upper=3.14 effort=10 velocity=2
- joint joint4_pitch: limit lower=-1.57 upper=1.57 effort=10 velocity=2 -> lower=-3.14 upper=3.14 effort=10 velocity=2
- joint joint4_yaw: limit lower=-1.57 upper=1.57 effort=10 velocity=2 -> lower=-3.14 upper=3.14 effort=10 velocity=2
- joint joint5_pitch: limit lower=-1.57 upper=1.57 effort=10 velocity=2 -> lower=-3.14 upper=3.14 effort=10 velocity=2
- joint joint5_yaw: limit lower=-1.57 upper=1.57 effort=10 velocity=2 -> lower=-3.14 upper=3.14 effort=10 velocity=2
- joint joint6_pitch: limit lower=-1.57 upper=1.57 effort=10 velocity=2 -> lower=-3.14 upper=3.14 effort=10 velocity=2
- joint joint6_yaw: limit lower=-1.57 upper=1.57 effort=10 velocity=2 -> lower=-3.14 upper=3.14 effort=10 velocity=2
- joint joint7_pitch: limit lower=-1.57 upper=1.57 effort=10 velocity=2 -> lower=-3.14 upper=3.14 effort=10 velocity=2
- joint joint7_yaw: limit lower=-1.57 upper=1.57 effort=10 velocity=2 -> lower=-3.14 upper=3.14 effort=10 velocity=2
