Commit message: CoG convergence

File: dragon.urdf (robot description, URDF)
Before this commit: robot L1, 26 links, 25 joints
Links:
- link F1: mass 0.05 -> 0
- link F2: mass 0.05 -> 0
- link F3: mass 0.05 -> 0
- link F4: mass 0.05 -> 0
- link G1: mass 0.05 -> 1
- link G2: mass 0.05 -> 1
- link G3: mass 0.05 -> 1
- link G4: mass 0.05 -> 1
- link L1: mass 0.01 -> 0
- link L1_rotor_L: mass 0.02 -> 0
- link L1_rotor_R: mass 0.02 -> 0
- link L2: mass 0.01 -> 0
- link L2_rotor_L: mass 0.02 -> 0
- link L2_rotor_R: mass 0.02 -> 0
- link L3: mass 0.01 -> 0
- link L3_rotor_L: mass 0.02 -> 0
- link L3_rotor_R: mass 0.02 -> 0
- link L4: mass 0.01 -> 0
- link L4_rotor_L: mass 0.02 -> 0
- link L4_rotor_R: mass 0.02 -> 0
- link joint1_pitch_link: mass 0.01 -> 0
- link joint1_yaw_link: mass 0.01 -> 0
- link joint2_pitch_link: mass 0.01 -> 0
- link joint2_yaw_link: mass 0.01 -> 0
- link joint3_pitch_link: mass 0.01 -> 0
- link joint3_yaw_link: mass 0.01 -> 0

Commit message: Force convergence

File: dragon.urdf (robot description, URDF)
Before this commit: robot L1, 26 links, 25 joints
Links:
- link F1: mass 0 -> 0.05
- link F2: mass 0 -> 0.05
- link F3: mass 0 -> 0.05
- link F4: mass 0 -> 0.05
- link G1: mass 1 -> 0.05
- link G2: mass 1 -> 0.05
- link G3: mass 1 -> 0.05
- link G4: mass 1 -> 0.05
- link L1: mass 0 -> 0.01
- link L1_rotor_L: mass 0 -> 0.02
- link L1_rotor_R: mass 0 -> 0.02
- link L2: mass 0 -> 0.01
- link L2_rotor_L: mass 0 -> 0.02
- link L2_rotor_R: mass 0 -> 0.02
- link L3: mass 0 -> 0.01
- link L3_rotor_L: mass 0 -> 0.02
- link L3_rotor_R: mass 0 -> 0.02
- link L4: mass 0 -> 0.01
- link L4_rotor_L: mass 0 -> 0.02
- link L4_rotor_R: mass 0 -> 0.02
- link joint1_pitch_link: mass 0 -> 0.01
- link joint1_yaw_link: mass 0 -> 0.01
- link joint2_pitch_link: mass 0 -> 0.01
- link joint2_yaw_link: mass 0 -> 0.01
- link joint3_pitch_link: mass 0 -> 0.01
- link joint3_yaw_link: mass 0 -> 0.01

Commit message: Improved COG

File: dragon.urdf (robot description, URDF)
Before this commit: robot L1, 26 links, 25 joints
Links:
- link L1: mass 0.01 -> 0.000000000000000001
- link L2: mass 0.01 -> 0.000000000000000001
- link L3: mass 0.01 -> 0.000000000000000001
- link L4: mass 0.01 -> 0.000000000000000001
- link joint1_pitch_link: mass 0.01 -> 0.000000000000000001
- link joint1_yaw_link: mass 0.01 -> 0.000000000000000001
- link joint2_pitch_link: mass 0.01 -> 0.000000000000000001
- link joint2_yaw_link: mass 0.01 -> 0.000000000000000001
- link joint3_pitch_link: mass 0.01 -> 0.000000000000000001
- link joint3_yaw_link: mass 0.01 -> 0.000000000000000001

Commit message: Updates

File: dragon.urdf (robot description, URDF)
Before this commit: robot L1, 26 links, 25 joints
Links:
- link L1: mass 0.000000000000000001 -> 0.01
- link L2: mass 0.000000000000000001 -> 0.01
- link L3: mass 0.000000000000000001 -> 0.01
- link L4: mass 0.000000000000000001 -> 0.01
- link joint1_pitch_link: mass 0.000000000000000001 -> 0.01
- link joint1_yaw_link: mass 0.000000000000000001 -> 0.01
- link joint2_pitch_link: mass 0.000000000000000001 -> 0.01
- link joint2_yaw_link: mass 0.000000000000000001 -> 0.01
- link joint3_pitch_link: mass 0.000000000000000001 -> 0.01
- link joint3_yaw_link: mass 0.000000000000000001 -> 0.01
Joints:
- joint L1_rotor_L_fix: origin xyz=0 0.15 0 rpy=0 0 0 -> xyz=0 0.1 0 rpy=0 0 0
- joint L1_rotor_R_fix: origin xyz=0 -0.15 0 rpy=0 0 0 -> xyz=0 -0.1 0 rpy=0 0 0
- joint L2_rotor_L_fix: origin xyz=0 0.15 0 rpy=0 0 0 -> xyz=0 0.1 0 rpy=0 0 0
- joint L2_rotor_R_fix: origin xyz=0 -0.15 0 rpy=0 0 0 -> xyz=0 -0.1 0 rpy=0 0 0
- joint L3_rotor_L_fix: origin xyz=0 0.15 0 rpy=0 0 0 -> xyz=0 0.1 0 rpy=0 0 0
- joint L3_rotor_R_fix: origin xyz=0 -0.15 0 rpy=0 0 0 -> xyz=0 -0.1 0 rpy=0 0 0
- joint L4_rotor_L_fix: origin xyz=0 0.15 0 rpy=0 0 0 -> xyz=0 0.1 0 rpy=0 0 0
- joint L4_rotor_R_fix: origin xyz=0 -0.15 0 rpy=0 0 0 -> xyz=0 -0.1 0 rpy=0 0 0

Commit message: Added anchors

File: dragon.urdf (robot description, URDF)
Before this commit: robot L1, 26 links, 25 joints
Links:
- added link joint0_yaw_link, mass 0.01; collision sphere radius=0.025
- added link joint4_yaw_link, mass 0.01; collision sphere radius=0.025
Joints:
- added joint joint0_yaw: type fixed, parent joint0_yaw_link, child L1, origin xyz=0.025 0 0 rpy=0 0 0
- added joint joint4_yaw: type fixed, parent L4, child joint4_yaw_link, origin xyz=0.325 0 0 rpy=0 0 0
