Commit message: Changed URDF to match ell = 1

File: assets/dragon.urdf (robot description, URDF)
Before this commit: robot joint0_yaw_link, 28 links, 27 joints
Links:
- link F1: geometry collision box size=0.1 0.50 0.01; collision cylinder length=0.01 radius=0.12
- link F2: geometry collision box size=0.1 0.50 0.01; collision cylinder length=0.01 radius=0.12
- link F3: geometry collision box size=0.1 0.50 0.01; collision cylinder length=0.01 radius=0.12
- link F4: geometry collision box size=0.1 0.50 0.01; collision cylinder length=0.01 radius=0.12
- link G1: geometry collision box size=0.86 0.1 0.1
- link G2: geometry collision box size=0.86 0.1 0.1
- link G3: geometry collision box size=0.86 0.1 0.1
- link G4: geometry collision box size=0.86 0.1 0.1
- link joint0_yaw_link: geometry collision sphere radius=0.07
- link joint1_yaw_link: geometry collision sphere radius=0.07
- link joint2_yaw_link: geometry collision sphere radius=0.07
- link joint3_yaw_link: geometry collision sphere radius=0.07
- link joint4_yaw_link: geometry collision sphere radius=0.07
Joints:
- joint L1_rotor_L_fix: origin xyz=0 0.1 0 rpy=0 0 0 -> xyz=0 0.2 0 rpy=0 0 0
- joint L1_rotor_R_fix: origin xyz=0 -0.1 0 rpy=0 0 0 -> xyz=0 -0.2 0 rpy=0 0 0
- joint L1_vec_phi: origin xyz=0.15 0 0 rpy=0 0 0 -> xyz=0.43 0 0 rpy=0 0 0
- joint L2_rotor_L_fix: origin xyz=0 0.1 0 rpy=0 0 0 -> xyz=0 0.2 0 rpy=0 0 0
- joint L2_rotor_R_fix: origin xyz=0 -0.1 0 rpy=0 0 0 -> xyz=0 -0.2 0 rpy=0 0 0
- joint L2_vec_phi: origin xyz=0.15 0 0 rpy=0 0 0 -> xyz=0.43 0 0 rpy=0 0 0
- joint L3_rotor_L_fix: origin xyz=0 0.1 0 rpy=0 0 0 -> xyz=0 0.2 0 rpy=0 0 0
- joint L3_rotor_R_fix: origin xyz=0 -0.1 0 rpy=0 0 0 -> xyz=0 -0.2 0 rpy=0 0 0
- joint L3_vec_phi: origin xyz=0.15 0 0 rpy=0 0 0 -> xyz=0.43 0 0 rpy=0 0 0
- joint L4_rotor_L_fix: origin xyz=0 0.1 0 rpy=0 0 0 -> xyz=0 0.2 0 rpy=0 0 0
- joint L4_rotor_R_fix: origin xyz=0 -0.1 0 rpy=0 0 0 -> xyz=0 -0.2 0 rpy=0 0 0
- joint L4_vec_phi: origin xyz=0.15 0 0 rpy=0 0 0 -> xyz=0.43 0 0 rpy=0 0 0
- joint joint0_yaw: origin xyz=0.025 0 0 rpy=0 0 0 -> xyz=0.07 0 0 rpy=0 0 0
- joint joint1_fix: origin xyz=0.025 0 0 rpy=0 0 0 -> xyz=0.07 0 0 rpy=0 0 0
- joint joint1_yaw: origin xyz=0.325 0 0 rpy=0 0 0 -> xyz=0.93 0 0 rpy=0 0 0
- joint joint2_fix: origin xyz=0.025 0 0 rpy=0 0 0 -> xyz=0.07 0 0 rpy=0 0 0
- joint joint2_yaw: origin xyz=0.325 0 0 rpy=0 0 0 -> xyz=0.93 0 0 rpy=0 0 0
- joint joint3_fix: origin xyz=0.025 0 0 rpy=0 0 0 -> xyz=0.07 0 0 rpy=0 0 0
- joint joint3_yaw: origin xyz=0.325 0 0 rpy=0 0 0 -> xyz=0.93 0 0 rpy=0 0 0
- joint joint4_yaw: origin xyz=0.325 0 0 rpy=0 0 0 -> xyz=0.93 0 0 rpy=0 0 0

File: assets/dragon_long.urdf (robot description, URDF)
Before this commit: robot L1, 54 links, 53 joints
Links:
- added link joint0_yaw_link, mass 0.01; collision sphere radius=0.07
- added link joint8_yaw_link, mass 0.01; collision sphere radius=0.07
- link F1: geometry collision box size=0.1 0.50 0.01; collision cylinder length=0.01 radius=0.12
- link F2: geometry collision box size=0.1 0.50 0.01; collision cylinder length=0.01 radius=0.12
- link F3: geometry collision box size=0.1 0.50 0.01; collision cylinder length=0.01 radius=0.12
- link F4: geometry collision box size=0.1 0.50 0.01; collision cylinder length=0.01 radius=0.12
- link F5: geometry collision box size=0.1 0.50 0.01; collision cylinder length=0.01 radius=0.12
- link F6: geometry collision box size=0.1 0.50 0.01; collision cylinder length=0.01 radius=0.12
- link F7: geometry collision box size=0.1 0.50 0.01; collision cylinder length=0.01 radius=0.12
- link F8: geometry collision box size=0.1 0.50 0.01; collision cylinder length=0.01 radius=0.12
- link G1: geometry collision box size=0.86 0.1 0.1
- link G2: geometry collision box size=0.86 0.1 0.1
- link G3: geometry collision box size=0.86 0.1 0.1
- link G4: geometry collision box size=0.86 0.1 0.1
- link G5: geometry collision box size=0.86 0.1 0.1
- link G6: geometry collision box size=0.86 0.1 0.1
- link G7: geometry collision box size=0.86 0.1 0.1
- link G8: geometry collision box size=0.86 0.1 0.1
- link L1: mass 0.000000000000000001 -> 0.001
- link L2: mass 0.000000000000000001 -> 0.001
- link L3: mass 0.000000000000000001 -> 0.001
- link L4: mass 0.000000000000000001 -> 0.001
- link L5: mass 0.000000000000000001 -> 0.001
- link L6: mass 0.000000000000000001 -> 0.001
- link L7: mass 0.000000000000000001 -> 0.001
- link L8: mass 0.000000000000000001 -> 0.001
- link joint1_pitch_link: mass 0.000000000000000001 -> 0.001
- link joint1_yaw_link: mass 0.000000000000000001 -> 0.001; geometry collision sphere radius=0.07
- link joint2_pitch_link: mass 0.000000000000000001 -> 0.001
- link joint2_yaw_link: mass 0.000000000000000001 -> 0.001; geometry collision sphere radius=0.07
- link joint3_pitch_link: mass 0.000000000000000001 -> 0.001
- link joint3_yaw_link: mass 0.000000000000000001 -> 0.001; geometry collision sphere radius=0.07
- link joint4_pitch_link: mass 0.000000000000000001 -> 0.001
- link joint4_yaw_link: mass 0.000000000000000001 -> 0.001; geometry collision sphere radius=0.07
- link joint5_pitch_link: mass 0.000000000000000001 -> 0.001
- link joint5_yaw_link: mass 0.000000000000000001 -> 0.001; geometry collision sphere radius=0.07
- link joint6_pitch_link: mass 0.000000000000000001 -> 0.001
- link joint6_yaw_link: mass 0.000000000000000001 -> 0.001; geometry collision sphere radius=0.07
- link joint7_pitch_link: mass 0.000000000000000001 -> 0.001
- link joint7_yaw_link: mass 0.000000000000000001 -> 0.001; geometry collision sphere radius=0.07
Joints:
- added joint joint0_yaw: type fixed, parent joint0_yaw_link, child L1, origin xyz=0.07 0 0 rpy=0 0 0
- added joint joint8_yaw: type fixed, parent L8, child joint8_yaw_link, origin xyz=0.93 0 0 rpy=0 0 0
- joint L1_rotor_L_fix: origin xyz=0 0.15 0 rpy=0 0 0 -> xyz=0 0.2 0 rpy=0 0 0
- joint L1_rotor_R_fix: origin xyz=0 -0.15 0 rpy=0 0 0 -> xyz=0 -0.2 0 rpy=0 0 0
- joint L1_vec_phi: origin xyz=0.15 0 0 rpy=0 0 0 -> xyz=0.43 0 0 rpy=0 0 0
- joint L2_rotor_L_fix: origin xyz=0 0.15 0 rpy=0 0 0 -> xyz=0 0.2 0 rpy=0 0 0
- joint L2_rotor_R_fix: origin xyz=0 -0.15 0 rpy=0 0 0 -> xyz=0 -0.2 0 rpy=0 0 0
- joint L2_vec_phi: origin xyz=0.15 0 0 rpy=0 0 0 -> xyz=0.43 0 0 rpy=0 0 0
- joint L3_rotor_L_fix: origin xyz=0 0.15 0 rpy=0 0 0 -> xyz=0 0.2 0 rpy=0 0 0
- joint L3_rotor_R_fix: origin xyz=0 -0.15 0 rpy=0 0 0 -> xyz=0 -0.2 0 rpy=0 0 0
- joint L3_vec_phi: origin xyz=0.15 0 0 rpy=0 0 0 -> xyz=0.43 0 0 rpy=0 0 0
- joint L4_rotor_L_fix: origin xyz=0 0.15 0 rpy=0 0 0 -> xyz=0 0.2 0 rpy=0 0 0
- joint L4_rotor_R_fix: origin xyz=0 -0.15 0 rpy=0 0 0 -> xyz=0 -0.2 0 rpy=0 0 0
- joint L4_vec_phi: origin xyz=0.15 0 0 rpy=0 0 0 -> xyz=0.43 0 0 rpy=0 0 0
- joint L5_rotor_L_fix: origin xyz=0 0.15 0 rpy=0 0 0 -> xyz=0 0.2 0 rpy=0 0 0
- joint L5_rotor_R_fix: origin xyz=0 -0.15 0 rpy=0 0 0 -> xyz=0 -0.2 0 rpy=0 0 0
- joint L5_vec_phi: origin xyz=0.15 0 0 rpy=0 0 0 -> xyz=0.43 0 0 rpy=0 0 0
- joint L6_rotor_L_fix: origin xyz=0 0.15 0 rpy=0 0 0 -> xyz=0 0.2 0 rpy=0 0 0
- joint L6_rotor_R_fix: origin xyz=0 -0.15 0 rpy=0 0 0 -> xyz=0 -0.2 0 rpy=0 0 0
- joint L6_vec_phi: origin xyz=0.15 0 0 rpy=0 0 0 -> xyz=0.43 0 0 rpy=0 0 0
- joint L7_rotor_L_fix: origin xyz=0 0.15 0 rpy=0 0 0 -> xyz=0 0.2 0 rpy=0 0 0
- joint L7_rotor_R_fix: origin xyz=0 -0.15 0 rpy=0 0 0 -> xyz=0 -0.2 0 rpy=0 0 0
- joint L7_vec_phi: origin xyz=0.15 0 0 rpy=0 0 0 -> xyz=0.43 0 0 rpy=0 0 0
- joint L8_rotor_L_fix: origin xyz=0 0.15 0 rpy=0 0 0 -> xyz=0 0.2 0 rpy=0 0 0
- joint L8_rotor_R_fix: origin xyz=0 -0.15 0 rpy=0 0 0 -> xyz=0 -0.2 0 rpy=0 0 0
- joint L8_vec_phi: origin xyz=0.15 0 0 rpy=0 0 0 -> xyz=0.43 0 0 rpy=0 0 0
- joint joint1_fix: origin xyz=0.025 0 0 rpy=0 0 0 -> xyz=0.07 0 0 rpy=0 0 0
- joint joint1_yaw: origin xyz=0.325 0 0 rpy=0 0 0 -> xyz=0.93 0 0 rpy=0 0 0
- joint joint2_fix: origin xyz=0.025 0 0 rpy=0 0 0 -> xyz=0.07 0 0 rpy=0 0 0
- joint joint2_yaw: origin xyz=0.325 0 0 rpy=0 0 0 -> xyz=0.93 0 0 rpy=0 0 0
- joint joint3_fix: origin xyz=0.025 0 0 rpy=0 0 0 -> xyz=0.07 0 0 rpy=0 0 0
- joint joint3_yaw: origin xyz=0.325 0 0 rpy=0 0 0 -> xyz=0.93 0 0 rpy=0 0 0
- joint joint4_fix: origin xyz=0.025 0 0 rpy=0 0 0 -> xyz=0.07 0 0 rpy=0 0 0
- joint joint4_yaw: origin xyz=0.325 0 0 rpy=0 0 0 -> xyz=0.93 0 0 rpy=0 0 0
- joint joint5_fix: origin xyz=0.025 0 0 rpy=0 0 0 -> xyz=0.07 0 0 rpy=0 0 0
- joint joint5_yaw: origin xyz=0.325 0 0 rpy=0 0 0 -> xyz=0.93 0 0 rpy=0 0 0
- joint joint6_fix: origin xyz=0.025 0 0 rpy=0 0 0 -> xyz=0.07 0 0 rpy=0 0 0
- joint joint6_yaw: origin xyz=0.325 0 0 rpy=0 0 0 -> xyz=0.93 0 0 rpy=0 0 0
- joint joint7_fix: origin xyz=0.025 0 0 rpy=0 0 0 -> xyz=0.07 0 0 rpy=0 0 0
- joint joint7_yaw: origin xyz=0.325 0 0 rpy=0 0 0 -> xyz=0.93 0 0 rpy=0 0 0

Commit message: Larger font

File: assets/dragon.urdf (robot description, URDF)
Before this commit: robot joint0_yaw_link, 28 links, 27 joints
Links:
- link L1: mass 0.01 -> 0.00000000001
- link L2: mass 0.01 -> 0.00000000001
- link L3: mass 0.01 -> 0.00000000001
- link L4: mass 0.01 -> 0.00000000001
- link joint0_yaw_link: mass 0.01 -> 0.00000000001
- link joint1_pitch_link: mass 0.01 -> 0.00000000001
- link joint1_yaw_link: mass 0.01 -> 0.00000000001
- link joint2_pitch_link: mass 0.01 -> 0.00000000001
- link joint2_yaw_link: mass 0.01 -> 0.00000000001
- link joint3_pitch_link: mass 0.01 -> 0.00000000001
- link joint3_yaw_link: mass 0.01 -> 0.00000000001
- link joint4_yaw_link: mass 0.01 -> 0.00000000001
