Commit message: Wrench simulations

File: assets/dragon_long.urdf (robot description, URDF)
Before this commit: robot joint0_yaw_link, 56 links, 55 joints
Links:
- link L1: mass 0.001 -> 0.00000000001
- link L2: mass 0.001 -> 0.00000000001
- link L3: mass 0.001 -> 0.00000000001
- link L4: mass 0.001 -> 0.00000000001
- link L5: mass 0.001 -> 0.00000000001
- link L6: mass 0.001 -> 0.00000000001
- link L7: mass 0.001 -> 0.00000000001
- link L8: mass 0.001 -> 0.00000000001
- link joint0_yaw_link: mass 0.01 -> 0.00000000001
- link joint1_pitch_link: mass 0.001 -> 0.00000000001
- link joint1_yaw_link: mass 0.001 -> 0.00000000001
- link joint2_pitch_link: mass 0.001 -> 0.00000000001
- link joint2_yaw_link: mass 0.001 -> 0.00000000001
- link joint3_pitch_link: mass 0.001 -> 0.00000000001
- link joint3_yaw_link: mass 0.001 -> 0.00000000001
- link joint4_pitch_link: mass 0.001 -> 0.00000000001
- link joint4_yaw_link: mass 0.001 -> 0.00000000001
- link joint5_pitch_link: mass 0.001 -> 0.00000000001
- link joint5_yaw_link: mass 0.001 -> 0.00000000001
- link joint6_pitch_link: mass 0.001 -> 0.00000000001
- link joint6_yaw_link: mass 0.001 -> 0.00000000001
- link joint7_pitch_link: mass 0.001 -> 0.00000000001
- link joint7_yaw_link: mass 0.001 -> 0.00000000001
- link joint8_yaw_link: mass 0.01 -> 0.00000000001
